File: Power - Charging .kicad_sch (KiCad schematic)
At the start: 0 parts

Commit message: added li-pol input, start creating charging circuit
Parts:
- added C37, C39: 4.7uF, 0_capacitors:C_0805_2012Metric, symbol 0_capacitors:CL21A475KAQNNNE
- added C38, C41: 100nF, 0_capacitors:C_0402_1005Metric, symbol 0_capacitors:CL05B104KO5NNNC
- added C42: 10uF, 0_capacitors:C_0805_2012Metric, symbol 0_capacitors:CL21A106KAYNNNE
- added R47, R48, R49: 10kΩ, 0_resistors:R_0402_1005Metric, symbol 0_resistors:0402WGF1002TCE
- added R50: 0Ω, 0_resistors:R_0402_1005Metric, symbol 0_resistors:0402WGF0000TCE
- added U3: MP2667GG-0000-Z, 0_integrated_circuits:QFN-10_2MMx2MM_MNP-L, symbol 0_integrated_circuits:MP2667GG-0000-Z
Connections:
- new net: R49.2, U3.3 (INT)
- new net: R47.1, R48.2, R50.2, U3.2 (NTC)
- new net: C38.1, U3.4 (VDD)
- new net +BATT: C42.1, U3.8 (BATT), U3.9 (BATT)
- new net GND: C37.2, C38.2, C39.2, C41.2, C42.2, R47.2, U3.5 (GND)
- new net NTC_BATT: R50.1
- new net VBUS: C37.1, R48.1, U3.1 (IN)
- new net VSYS: C39.1, C41.1, U3.10 (SYS)
Other:
- title: (none) -> Power - Charging
