File: LCD.kicad_sch (KiCad schematic)
At the start: 41 parts, among them J1 AFC07-S40ECA-00, J11 AFC07-S10FCC-00

Commit message: designator chagnes and cleanup silkscreen
Parts:
- C10, C11, C9: LCSC PN (none) -> C1525
- C12, C13: LCSC PN (none) -> C1779
- J1: LCSC PN (none) -> C262648
- J11: LCSC PN (none) -> C11050
- R7, R8: LCSC PN (none) -> C25744
Changed lines of the file:
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@@
 			)
 		)
+		(property "LCSC PN" "C1525"
+			(at 144.78 186.69 0)
+			(effects
+				(font
+					(size 1.27 1.27)
+				)
+				(hide yes)
+			)
+		)
 		(pin "2"
 		)
@@
 			)
 		)
-		(property "Description" "Resistor, small symbol"
+		(property "Description" "50V ±100ppm/℃ ±1% 10kΩ 0402"
 			(at 134.62 92.71 0)
 			(effects
@@
 			)
 		)
+		(property "LCSC PN" "C25744"
+			(at 134.62 92.71 0)
+			(effects
+				(font
+					(size 1.27 1.27)
+				)
+				(hide yes)
+			)
+		)
 		(pin "2"
 		)
@@
 			)
 		)
+		(property "LCSC PN" "C262648"
+			(at 271.78 39.37 0)
+			(effects
+				(font
+					(size 1.27 1.27)
+				)
+				(hide yes)
+			)
+		)
 		(pin "14"
 		)
@@
 			)
 		)
+		(property "LCSC PN" "C1525"
+			(at 134.62 101.6 0)
+			(effects
+				(font
+					(size 1.27 1.27)
+				)
+				(hide yes)
+			)
+		)
 		(pin "1"
 		)
@@
 			)
 		)
+		(property "LCSC PN" "C1779"
+			(at 134.62 44.45 0)
+			(effects
+				(font
+					(size 1.27 1.27)
+				)
+				(hide yes)
+			)
+		)
 		(pin "2"
 		)
@@
 			)
 		)
+		(property "LCSC PN" "C11050"
+			(at 271.78 208.28 0)
+			(effects
+				(font
+					(size 1.27 1.27)
+				)
+				(hide yes)
+			)
+		)
 		(pin "7"
 		)
@@
 			)
 		)
-		(property "Description" "Resistor, small symbol"
+		(property "Description" "50V ±100ppm/℃ ±1% 10kΩ 0402"
 			(at 134.62 217.17 0)
 			(effects
@@
 			)
 		)
+		(property "LCSC PN" "C25744"
+			(at 134.62 217.17 0)
+			(effects
+				(font
+					(size 1.27 1.27)
+				)
+				(hide yes)
+			)
+		)
 		(pin "2"
 		)
@@
 			)
 		)
+		(property "LCSC PN" "C1525"
+			(at 144.78 44.45 0)
+			(effects
+				(font
+					(size 1.27 1.27)
+				)
+				(hide yes)
+			)
+		)
 		(pin "2"
 		)
@@
 			(at 134.62 186.69 0)
 			(effects
+				(font
+					(size 1.27 1.27)
+				)
+				(hide yes)
+			)
+		)
+		(property "LCSC PN" "C1779"
+			(at 134.62 186.69 0)
+			(effects
