File: UI - Buzzer.kicad_sch (KiCad schematic)
At the start: 6 parts, among them Q4 AO3400A

Commit message: designator chagnes and cleanup silkscreen
Parts:
- D2: LCSC PN (none) -> C191023
- Q4: LCSC PN (none) -> C20917
- R75: LCSC PN (none) -> C25104
- R76: LCSC PN (none) -> C25792
Changed lines of the file:
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@@
+			)
+		)
+		(property "LCSC PN" "C25792"
+			(at 134.62 96.52 0)
+			(effects
+				(font
+					(size 1.27 1.27)
+				)
+				(hide yes)
 			)
 		)
@@
 			)
 		)
+		(property "LCSC PN" "C25104"
+			(at 127 87.63 0)
+			(effects
+				(font
+					(size 1.27 1.27)
+				)
+				(hide yes)
+			)
+		)
 		(pin "1"
 		)
@@
 			)
 		)
+		(property "LCSC PN" "C20917"
+			(at 144.78 87.63 0)
+			(effects
+				(font
+					(size 1.27 1.27)
+				)
+				(hide yes)
+			)
+		)
 		(pin "2"
 		)
@@
 			(at 133.35 73.66 0)
 			(effects
+				(font
+					(size 1.27 1.27)
+				)
+				(hide yes)
+			)
+		)
+		(property "LCSC PN" "C191023"
+			(at 133.35 73.66 0)
+			(effects
