File: auxiliary.kicad_sch (KiCad schematic)
At the start: 39 parts, among them J7 Conn_01x05, J9 Conn_02x06_Odd_Even, U6 PCA9554APW, Y1 32.768KHZ, Y2 X322525MOB4SI-25MHz

Commit message: designator chagnes and cleanup silkscreen
Parts:
- C79, C80: LCSC PN (none) -> C1525
- C81, C82, C83, C84: LCSC PN (none) -> C1576
- C85: LCSC PN (none) -> C15849
- J10, J8: footprint Connector_PinHeader_2.00mm:PinHeader_1x02_P2.00mm_Vertical -> Connector_PinHeader_2.54mm:PinHeader_1x02_P2.54mm_Vertical; LCSC PN (none) -> C492401; Supplier Part Number 1 C541856 -> C492401
- J7: LCSC PN (none) -> C157993
- R79, R84, R85, R86, R91, R92, R93, R94: LCSC PN (none) -> C25744
- R80, R81, R82, R83, R87, R88: LCSC PN (none) -> C17168
- R89, R90: LCSC PN (none) -> C25905
- U6: LCSC PN (none) -> C86803
- Y1: LCSC PN (none) -> C32346
- Y2: LCSC PN (none) -> C9006
